File: PCB/Smart Servo Breadboard Control Board Rev.2/Smart Servo Control Board Rev.2.kicad_pcb (KiCad board)
At the start: 4 copper layers, 120 x 120 mm, 72 parts, among them J1 ESP-L, J10 SCL, J11 SDA, J12 GND, J13 MOT1, J14 MOT, J15 MOT2, J16 OUT, J17 STLINK, J2 ESP-R, J3 STM-L, J4 STM-R, J5 5V, J6 SCL, J7 SDA, J8 GND, J9 5V, U1 AS5600, U2 24LC256, U3 INA219AxD, U4 INA219AxD, U5 AMS1117-3.3, U6 DRV8830DGQR, U7 STM32F103C8Tx

Commit message: Lugre and various tests
Parts:
- removed J12: GND, Connector_PinSocket_2.54mm:PinSocket_1x04_P2.54mm_Vertical
- removed J5: 5V, Connector_PinHeader_2.54mm:PinHeader_1x04_P2.54mm_Vertical
- removed J8: GND, Connector_PinHeader_2.54mm:PinHeader_1x04_P2.54mm_Vertical
- removed J9: 5V, Connector_PinSocket_2.54mm:PinSocket_1x04_P2.54mm_Vertical
- added D2: PWR, Diode_SMD:D_1206_3216Metric_Pad1.42x1.75mm_HandSolder, B.Cu at (245.0, 72.0)
- added R12: 1K, Resistor_SMD:R_0603_1608Metric_Pad0.98x0.95mm_HandSolder, B.Cu at (245.0, 77.0)
- C12, C3, C4, C5, C6, D1, J1, J10, J11, J2, J3, J4, R11, R2, R4, R6, R7, R8: moved to B.Cu
- C13, C14, C15, C16, J14, J6, J7: moved to F.Cu
- H1, H10, H11, H14, H15, H2, H3, H4, H5, H6, H7, H8: footprint MountingHole:MountingHole_3.2mm_M3 -> MountingHole:MountingHole_4.3mm_M4
- H12, H13, H16, H9: footprint MountingHole:MountingHole_3.2mm_M3 -> MountingHole:MountingHole_4.3mm_M4_DIN965_Pad_TopBottom
- J13, J15: footprint Connector_PinHeader_2.54mm:PinHeader_1x01_P2.54mm_Vertical -> TestPoint:TestPoint_Pad_3.0x3.0mm
- moved J6 144.8 mm to (248.8, 61.0), turned to -90 degrees
- moved J1 132.0 mm to (237.5, 49.7), turned to 180 degrees
- moved J3 125.2 mm to (233.7, 48.4), turned to 180 degrees
- moved H14 122.5 mm to (210.0, 42.5)
- moved H13 118.7 mm to (210.0, 102.5)
- moved J7 115.3 mm to (248.8, 66.0), turned to -90 degrees
- moved H15 104.1 mm to (240.0, 42.5)
- moved H16 99.6 mm to (240.0, 102.5)
- moved J4 99.1 mm to (218.4, 48.4), turned to 180 degrees
- moved J2 93.0 mm to (214.6, 49.7), turned to 180 degrees
- moved R8 90.4 mm to (195.0, 77.0), turned to -90 degrees
- moved D1 85.1 mm to (195.0, 72.0), turned to 90 degrees
- moved J10 83.9 mm to (198.8, 61.0), turned to 90 degrees
- moved H5 66.3 mm to (110.0, 102.5)
- moved H6 66.0 mm to (110.0, 42.5)
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Connections:
- J16 pad 2: SDA2 -> SCL2
- J16 pad 3: SCL2 -> SDA2
- J17 pad 2: SWCLK -> SWDIO
- J17 pad 3: SWDIO -> SWCLK
- U6 pad V: (no net) -> GNDD
- U7 pad 30: FAULT -> unconnected-(U7-Pad30)
- U7 pad 46: unconnected-(U7-Pad46) -> FAULT
Routing:
- net GNDD: track 19.9 -> 99.3 mm, vias 0 -> 11
- net SCL: track 8.86 -> 44.7 mm
- net +3V3: track 39.3 -> 74.5 mm, vias 0 -> 9
- net +5V: track 22.7 -> 55.1 mm, vias 1 -> 2
- net SDA2: track 1.24 -> 32.9 mm, vias 0 -> 1
- net SCL2: track 1.11 -> 31.0 mm, vias 0 -> 1
- net SDA: track 7.62 -> 30.3 mm
- net SDA1: track 55.5 -> 67.8 mm, vias 3 -> 4
- net SCL1: track 58.4 -> 66.9 mm, vias 2 -> 5
- net SWDIO: track 10.6 -> 2.89 mm
- net GND: track 7.62 -> 0.00 mm
- net 5V: track 7.62 -> 1.49 mm, vias 0 -> 1
- net H-Bridge 2: track 17.5 -> 12.8 mm
- net SWCLK: track 7.58 -> 4.36 mm
- net FAULT: track 9.45 -> 6.35 mm, vias 0 -> 1
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- added copper zone on F.Cu, net +3V3
- added copper zone on In2.Cu, net +3V3
- added copper zone on F.Cu, net +5V
- added copper zone on In2.Cu, net +5V
- added copper zone on F.Cu, net 5V
- added copper zone on In2.Cu, net 5V
- added copper zone on B.Cu, net GND
- added copper zone on In1.Cu, net GND
- added copper zone on B.Cu, net GNDD
- added copper zone on In1.Cu, net GNDD
Other:
- board size 120 x 120 mm -> 201 x 73 mm
- board text added: "DRV8830 0xC1"
- board text added: "USB PORT"
- board text removed: "+5V"
- board text removed: "GND"
- board text removed: "MOTOR"

Commit message: codice e scheda a buon punto
Parts:
- removed H1: 1A, MountingHole:MountingHole_4.3mm_M4
- removed H17: M1, MountingHole:MountingHole_3.2mm_M3
- removed H18: M2, MountingHole:MountingHole_3.2mm_M3
- removed H19: M3, MountingHole:MountingHole_3.2mm_M3
- removed H2: 1B, MountingHole:MountingHole_4.3mm_M4
- removed H20: M4, MountingHole:MountingHole_3.2mm_M3
- removed H3: 1C, MountingHole:MountingHole_4.3mm_M4
- removed H4: 1D, MountingHole:MountingHole_4.3mm_M4
- removed H5: 2A, MountingHole:MountingHole_4.3mm_M4
- removed H6: 2B, MountingHole:MountingHole_4.3mm_M4
- removed H7: 2C, MountingHole:MountingHole_4.3mm_M4
- removed H8: 2D, MountingHole:MountingHole_4.3mm_M4
- removed J10: SCL, Connector_PinSocket_2.54mm:PinSocket_1x04_P2.54mm_Vertical
- removed J11: SDA, Connector_PinSocket_2.54mm:PinSocket_1x04_P2.54mm_Vertical
- removed J13: MOT1, TestPoint:TestPoint_Pad_3.0x3.0mm
- removed J15: MOT2, TestPoint:TestPoint_Pad_3.0x3.0mm
- removed J16: OUT, Connector_PinHeader_2.54mm:PinHeader_1x04_P2.54mm_Vertical
- removed J17: STLINK, Connector_PinHeader_2.54mm:PinHeader_1x04_P2.54mm_Vertical
- removed J7: SDA, Connector_PinHeader_2.54mm:PinHeader_1x04_P2.54mm_Vertical
- added D3: FAULT, Diode_SMD:D_1206_3216Metric_Pad1.42x1.75mm_HandSolder, B.Cu at (199.5, 96.7)
- added D4: FAULT, Diode_SMD:D_1206_3216Metric_Pad1.42x1.75mm_HandSolder, B.Cu at (249.5, 96.7)
- added J5: Conn_02x20_Odd_Even, Connector_PinSocket_2.54mm:PinSocket_2x20_P2.54mm_Vertical, B.Cu at (243.7, 48.4)
- added R13: 10m, Resistor_SMD:R_0603_1608Metric_Pad0.98x0.95mm_HandSolder, F.Cu at (181.1, 95.7)
- added R14: 1K, Resistor_SMD:R_0603_1608Metric_Pad0.98x0.95mm_HandSolder, B.Cu at (249.5, 92.3)
- added U10: AH49E, Package_TO_SOT_SMD:SOT-23, F.Cu at (180.5, 78.6)
- added U11: AH49E, Package_TO_SOT_SMD:SOT-23, F.Cu at (180.5, 87.5)
- added U8: AH49E, Package_TO_SOT_THT:TO-92S, F.Cu at (173.1, 87.8)
- added U9: AH49E, Package_TO_SOT_THT:TO-92S, F.Cu at (171.3, 80.1)
- C10, C11, C12, C2, C3, C4, C5, C6, C8, C9, R2, R4, R6, U5, U7: moved to F.Cu
- J6: value SCL -> Conn_02x20_Odd_Even; footprint Connector_PinHeader_2.54mm:PinHeader_1x04_P2.54mm_Vertical -> Connector_PinSocket_2.54mm:PinSocket_2x20_P2.54mm_Vertical; moved to B.Cu
- R11: value 10K -> 1K
- R5: moved to B.Cu
- R7: value 10m -> 220K; moved to F.Cu
- U3, U4: footprint Package_SO:SO-8_3.9x4.9mm_P1.27mm -> Package_SO:SOIC-8_3.9x4.9mm_P1.27mm
- moved J6 56.5 mm to (193.7, 48.4), turned to 180 degrees
- moved R10 37.5 mm to (199.5, 60.5), turned to 90 degrees
- moved U6 34.9 mm to (176.0, 104.0), turned to -90 degrees
- moved C4 34.2 mm to (189.4, 97.0), turned to 90 degrees
- moved C3 32.8 mm to (162.7, 97.0), turned to -90 degrees
- moved R11 31.8 mm to (199.5, 92.3), turned to 90 degrees
- moved C7 31.8 mm to (173.5, 104.0), turned to -90 degrees
- moved U4 31.0 mm to (185.6, 97.0), turned to 90 degrees
- moved U3 31.0 mm to (166.5, 97.0)
- moved R9 28.5 mm to (199.5, 64.3)
- moved U2 27.5 mm to (158.3, 76.7), turned to 0 degrees
- moved R1 27.4 mm to (171.0, 100.2), turned to 180 degrees
- moved C11 26.7 mm to (155.7, 83.7), turned to 180 degrees
- moved R5 26.3 mm to (171.0, 100.6), turned to -90 degrees
- moved C2 26.2 mm to (158.3, 72.9)
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Connections:
- net ISENSE renamed Net-(R5-Pad1)
- J14 pad 1: I_SENS_1 - -> I_SENS_2 -
- J14 pad 2: I_SENS_2 - -> I_SENS_1 -
- J6 pad 1: SCL -> GNDD
- J6 pad 2: SCL -> GNDD
- J6 pad 3: SCL -> +5V
- J6 pad 4: SCL -> +5V
- R10 pad 1: SDA1 -> +3V3
- R10 pad 2: +3V3 -> SDA2
- R11 pad 1: FAULT -> Net-(D3-Pad2)
- R6 pad 1: H-Bridge 1 -> I_SENS_1 -
- R6 pad 2: I_SENS_1 - -> H-Bridge 1
- R7 pad 1: I_SENS_2 - -> H-Bridge 2
- R7 pad 2: H-Bridge 2 -> H-Bridge 1
- R9 pad 1: SCL1 -> +3V3
- R9 pad 2: +3V3 -> SCL2
- U1 pad 6: SDA1 -> SDA2
- U1 pad 7: SCL1 -> SCL2
- U2 pad 5: SDA1 -> SDA2
- U2 pad 6: SCL1 -> SCL2
- U3 pad 3: SDA1 -> SDA2
- U3 pad 4: SCL1 -> SCL2
- U4 pad 3: SDA1 -> SDA2
- U4 pad 4: SCL1 -> SCL2
- U6 pad 10: SCL1 -> SCL2
- U6 pad 9: SDA1 -> SDA2
- U7 pad 21: SCL2 -> SCL1
- U7 pad 22: SDA2 -> SDA1
- U7 pad 42: SCL1 -> SCL2
- U7 pad 43: SDA1 -> SDA2
Routing:
- net +3V3: track 74.5 -> 191.1 mm, vias 9 -> 3
- net SCL2: track 31.0 -> 121.6 mm, vias 1 -> 4
- net GNDD: track 99.3 -> 14.3 mm, vias 11 -> 1
- net FAULT: track 6.35 -> 86.9 mm, vias 1 -> 2
- net SDA2: track 32.9 -> 111.2 mm
- net +5V: track 55.1 -> 116.4 mm
- net Net-(J5-Pad5): track 0.00 -> 44.4 mm
- net SDA1: track 67.8 -> 24.2 mm, vias 4 -> 1
- net SCL1: track 66.9 -> 23.4 mm, vias 5 -> 1
- net H-Bridge 1: track 13.7 -> 53.2 mm, vias 2 -> 1
- net H-Bridge 2: track 12.8 -> 47.7 mm, vias 2 -> 3
- net 49E_1: track 0.00 -> 34.7 mm
- net 49E_2: track 0.00 -> 25.0 mm
- net SWDIO: track 2.89 -> 26.3 mm, vias 0 -> 1
- net SWCLK: track 4.36 -> 25.6 mm, vias 0 -> 1
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- added copper zone on F.Cu, net GNDD
- removed copper zone on In2.Cu, net +3V3
- removed copper zone on In2.Cu, net +5V
- removed copper zone on In2.Cu, net 5V
- removed copper zone on In1.Cu, net GND
- removed copper zone on In1.Cu, net GNDD
Other:
- board size 201 x 73 mm -> 100 x 73 mm
- board text added: "+3.3V"
- board text added: "+5V"
- board text added: "49E-1"
- board text added: "49E-2"
- board text added: "49E-3"
- board text added: "49E-4"
- board text added: "DRV-1"
- board text added: "DRV-2"
- board text added: "ESP32 or STM32"
- board text added: "FAULT"
- board text added: "GND"
- board text added: "INA1 +"
- board text added: "INA1 -"
- board text added: "INA2 +"
- board text added: "INA2 -"
- board text added: "JLCJLCJLCJLC"
- board text added: "SCL1"
- board text added: "SCL2"
- board text added: "SDA1"
- board text added: "SDA2"
- board text added: "SWCLK"
- board text added: "SWDIO"
- board text removed: "2"
- board text removed: "24LC256 0x50"
- board text removed: "3"
- board text removed: "4"
- board text removed: "AS5600 0x36"
- board text removed: "DRV8830 0xC1"
- board text removed: "INA219-1 0x40"
- board text removed: "INA219-2 0x45"
- board text removed: "SCL"
- board text removed: "SDA"
