File: PCB/Smart Servo Breadboard Control Board Rev.2/Smart Servo Control Board Rev.2.kicad_sch (KiCad schematic)
At the start: 72 parts, among them J1 ESP-L, J10 SCL, J11 SDA, J12 GND, J13 MOT1, J14 MOT, J15 MOT2, J16 OUT, J17 STLINK, J2 ESP-R, J3 STM-L, J4 STM-R, J5 5V, J6 SCL, J7 SDA, J8 GND, J9 5V, U1 AS5600, U2 24LC256, U3 INA219AxD, U4 INA219AxD, U5 AMS1117-3.3, U6 DRV8830DGQR, U7 STM32F103C8Tx

Commit message: Lugre and various tests
Parts:
- removed H12: 3D, MountingHole:MountingHole_3.2mm_M3, symbol Mechanical:MountingHole
- removed H13: 4A, MountingHole:MountingHole_3.2mm_M3, symbol Mechanical:MountingHole
- removed H16: 4D, MountingHole:MountingHole_3.2mm_M3, symbol Mechanical:MountingHole
- removed H9: 3A, MountingHole:MountingHole_3.2mm_M3, symbol Mechanical:MountingHole
- removed J12: GND, Connector_PinSocket_2.54mm:PinSocket_1x04_P2.54mm_Vertical, symbol Connector:Conn_01x04_Female
- removed J5: 5V, Connector_PinHeader_2.54mm:PinHeader_1x04_P2.54mm_Vertical, symbol Connector:Conn_01x04_Male
- removed J8: GND, Connector_PinHeader_2.54mm:PinHeader_1x04_P2.54mm_Vertical, symbol Connector:Conn_01x04_Male
- removed J9: 5V, Connector_PinSocket_2.54mm:PinSocket_1x04_P2.54mm_Vertical, symbol Connector:Conn_01x04_Female
- added D2: PWR, Diode_SMD:D_1206_3216Metric_Pad1.42x1.75mm_HandSolder, symbol Device:LED
- added H12: 3D, MountingHole:MountingHole_4.3mm_M4_DIN965_Pad_TopBottom, symbol Mechanical:MountingHole_Pad
- added H13: 4A, MountingHole:MountingHole_4.3mm_M4_DIN965_Pad_TopBottom, symbol Mechanical:MountingHole_Pad
- added H16: 4D, MountingHole:MountingHole_4.3mm_M4_DIN965_Pad_TopBottom, symbol Mechanical:MountingHole_Pad
- added H9: 3A, MountingHole:MountingHole_4.3mm_M4_DIN965_Pad_TopBottom, symbol Mechanical:MountingHole_Pad
- added R12: 1K, Resistor_SMD:R_0603_1608Metric_Pad0.98x0.95mm_HandSolder, symbol Device:R
- H1, H10, H11, H14, H15, H2, H3, H4, H5, H6, H7, H8: footprint MountingHole:MountingHole_3.2mm_M3 -> MountingHole:MountingHole_4.3mm_M4
- J13, J15: footprint Connector_PinHeader_2.54mm:PinHeader_1x01_P2.54mm_Vertical -> TestPoint:TestPoint_Pad_3.0x3.0mm
Connections:
- net +5V: now also H9.1
- net 5V: now also D2.2 (A), H13.1
- net FAULT: now also U7.46 (PB9); no longer U7.30 (PA9)
- net GND: now also H16.1, R12.2
- net GNDD: now also H12.1
- net SCL2: now also J16.2 (Pin_2); no longer J16.3 (Pin_3)
- net SDA2: now also J16.3 (Pin_3); no longer J16.2 (Pin_2)
- net SWCLK: now also J17.3 (Pin_3); no longer J17.2 (Pin_2)
- net SWDIO: now also J17.2 (Pin_2); no longer J17.3 (Pin_3)
- new net: D2.1 (K), R12.1
Other:
- moved on the sheet: D1, H10, H11, H14, H15, J10, J11, J17, J6, J7, R8

Commit message: codice e scheda a buon punto
Parts:
- removed H1: 1A, MountingHole:MountingHole_4.3mm_M4, symbol Mechanical:MountingHole
- removed H17: M1, MountingHole:MountingHole_3.2mm_M3, symbol Mechanical:MountingHole
- removed H18: M2, MountingHole:MountingHole_3.2mm_M3, symbol Mechanical:MountingHole
- removed H19: M3, MountingHole:MountingHole_3.2mm_M3, symbol Mechanical:MountingHole
- removed H2: 1B, MountingHole:MountingHole_4.3mm_M4, symbol Mechanical:MountingHole
- removed H20: M4, MountingHole:MountingHole_3.2mm_M3, symbol Mechanical:MountingHole
- removed H3: 1C, MountingHole:MountingHole_4.3mm_M4, symbol Mechanical:MountingHole
- removed H4: 1D, MountingHole:MountingHole_4.3mm_M4, symbol Mechanical:MountingHole
- removed H5: 2A, MountingHole:MountingHole_4.3mm_M4, symbol Mechanical:MountingHole
- removed H6: 2B, MountingHole:MountingHole_4.3mm_M4, symbol Mechanical:MountingHole
- removed H7: 2C, MountingHole:MountingHole_4.3mm_M4, symbol Mechanical:MountingHole
- removed H8: 2D, MountingHole:MountingHole_4.3mm_M4, symbol Mechanical:MountingHole
- removed J10: SCL, Connector_PinSocket_2.54mm:PinSocket_1x04_P2.54mm_Vertical, symbol Connector:Conn_01x04_Female
- removed J11: SDA, Connector_PinSocket_2.54mm:PinSocket_1x04_P2.54mm_Vertical, symbol Connector:Conn_01x04_Female
- removed J13: MOT1, TestPoint:TestPoint_Pad_3.0x3.0mm, symbol Connector:Conn_01x01_Female
- removed J15: MOT2, TestPoint:TestPoint_Pad_3.0x3.0mm, symbol Connector:Conn_01x01_Female
- removed J16: OUT, Connector_PinHeader_2.54mm:PinHeader_1x04_P2.54mm_Vertical, symbol Connector:Conn_01x04_Female
- removed J17: STLINK, Connector_PinHeader_2.54mm:PinHeader_1x04_P2.54mm_Vertical, symbol Connector:Conn_01x04_Female
- removed J6: SCL, Connector_PinHeader_2.54mm:PinHeader_1x04_P2.54mm_Vertical, symbol Connector:Conn_01x04_Male
- removed J7: SDA, Connector_PinHeader_2.54mm:PinHeader_1x04_P2.54mm_Vertical, symbol Connector:Conn_01x04_Male
- added D3, D4: FAULT, Diode_SMD:D_1206_3216Metric_Pad1.42x1.75mm_HandSolder, symbol Device:LED
- added J5, J6: Conn_02x20_Odd_Even, Connector_PinSocket_2.54mm:PinSocket_2x20_P2.54mm_Vertical, symbol Connector_Generic:Conn_02x20_Odd_Even
- added R13: 10m, Resistor_SMD:R_0603_1608Metric_Pad0.98x0.95mm_HandSolder, symbol Device:R
- added R14: 1K, Resistor_SMD:R_0603_1608Metric_Pad0.98x0.95mm_HandSolder, symbol Device:R
- added U10, U11: AH49E, Package_TO_SOT_SMD:SOT-23, symbol Custom:AH49E
- added U8, U9: AH49E, Package_TO_SOT_THT:TO-92S, symbol Custom:AH49E
- R11: value 10K -> 1K
- R7: value 10m -> 220K
- U3, U4: footprint Package_SO:SO-8_3.9x4.9mm_P1.27mm -> Package_SO:SOIC-8_3.9x4.9mm_P1.27mm
Connections:
- net +3V3: now also R10.1, R9.1, J6.5 (Pin_5), J6.6 (Pin_6), U10.1 (VCC), U11.1 (VCC), U8.1 (VCC), U9.1 (VCC); no longer R10.2, R9.2
- net +5V: now also J6.3 (Pin_3), J6.4 (Pin_4)
- net 5V: now also J5.3 (Pin_3), J5.4 (Pin_4)
- net FAULT: now also D3.1 (K), J6.39 (Pin_39), J6.40 (Pin_40); no longer R11.1
- net GND: now also J5.1 (Pin_1), J5.2 (Pin_2)
- net GNDD: now also J6.1 (Pin_1), J6.2 (Pin_2), U10.2 (GND), U11.2 (GND), U8.2 (GND), U9.2 (GND)
- net H-Bridge 1: now also R6.2, R7.2, J6.27 (Pin_27), J6.28 (Pin_28), J6.31 (Pin_31), J6.32 (Pin_32); no longer R6.1
- net H-Bridge 2: now also R7.1, J6.29 (Pin_29), J6.30 (Pin_30), J6.37 (Pin_37), J6.38 (Pin_38), R13.2; no longer R7.2
- net I_SENS_1 -: now also J14.2 (Pin_2), R6.1, J6.33 (Pin_33), J6.34 (Pin_34); no longer J14.1 (Pin_1), R6.2
- net I_SENS_2 -: now also J14.1 (Pin_1), J6.35 (Pin_35), J6.36 (Pin_36), R13.1; no longer J14.2 (Pin_2), R7.1
- net SCL: now also J5.13 (Pin_13), J5.14 (Pin_14)
- net SCL1: now also U7.21 (PB10), J6.10 (Pin_10), J6.9 (Pin_9); no longer R9.1, U1.7 (SCL), U2.6 (SCL), U3.4 (SCL), U4.4 (SCL), U6.10 (SCL), U7.42 (PB6)
- net SCL2: now also R9.2, U1.7 (SCL), U2.6 (SCL), U3.4 (SCL), U4.4 (SCL), U6.10 (SCL), U7.42 (PB6), J6.13 (Pin_13), J6.14 (Pin_14); no longer U7.21 (PB10)
- net SDA: now also J5.11 (Pin_11), J5.12 (Pin_12)
- net SDA1: now also U7.22 (PB11), J6.7 (Pin_7), J6.8 (Pin_8); no longer R10.1, U1.6 (SDA), U2.5 (SDA), U3.3 (SDA), U4.3 (SDA), U6.9 (SDA), U7.43 (PB7)
- net SDA2: now also R10.2, U1.6 (SDA), U2.5 (SDA), U3.3 (SDA), U4.3 (SDA), U6.9 (SDA), U7.43 (PB7), J6.11 (Pin_11), J6.12 (Pin_12); no longer U7.22 (PB11)
- net SWCLK: now also J6.17 (Pin_17), J6.18 (Pin_18)
- net SWDIO: now also J6.15 (Pin_15), J6.16 (Pin_16)
- net ISENSE: no longer names the net of R5.1, U6.2 (ISENSE)
- new net: D3.2 (A), R11.1
- new net: D4.2 (A), R14.1
- new net: J5.5 (Pin_5), J5.6 (Pin_6), R14.2
- new net: D4.1 (K), J5.39 (Pin_39), J5.40 (Pin_40)
- new net: J5.10 (Pin_10), J5.9 (Pin_9)
- new net: J5.15 (Pin_15), J5.16 (Pin_16)
- new net: J5.17 (Pin_17), J5.18 (Pin_18)
- new net: J5.19 (Pin_19), J5.20 (Pin_20)
- new net: J5.21 (Pin_21), J5.22 (Pin_22)
- new net: J5.23 (Pin_23), J5.24 (Pin_24)
- new net: J5.25 (Pin_25), J5.26 (Pin_26)
- new net: J5.27 (Pin_27), J5.28 (Pin_28)
- new net: J5.29 (Pin_29), J5.30 (Pin_30)
- new net: J5.31 (Pin_31), J5.32 (Pin_32)
- new net: J5.33 (Pin_33), J5.34 (Pin_34)
- new net: J5.35 (Pin_35), J5.36 (Pin_36)
- new net: J5.37 (Pin_37), J5.38 (Pin_38)
- new net: J5.7 (Pin_7), J5.8 (Pin_8)
- new net 49E_1: J6.19 (Pin_19), J6.20 (Pin_20), U8.3 (OUT)
- new net 49E_2: J6.21 (Pin_21), J6.22 (Pin_22), U9.3 (OUT)
- new net 49E_3: J6.23 (Pin_23), J6.24 (Pin_24), U10.3 (OUT)
- new net 49E_4: J6.25 (Pin_25), J6.26 (Pin_26), U11.3 (OUT)
Other:
- note added: "CPU"
- note added: "Exerimental Speed Sensor"
- note added: "Motor & Driver"
- note added: "Position Sensor"
- note removed: "H-Bridge & Motor Connectors"
- note removed: "I2C Bus Pull-up Resistors"
- note removed: "Position Sensor Connector"
- moved on the sheet: C1, C10, C11, C12, C13, C14, C15, C16, C2, C7, C8, C9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
